File: smartdim.sch (EAGLE design)
At the start: 8 parts, among them Q1 N-HEXFET-2D_SOT232-, U1 Tiny85-20-SMT

Commit message: Remove unnecessary pullup
Parts:
- removed R1: 4K7, rcl:R-US_R0805
Connections:
- net +5V: no longer R1.2
- net USER_INPUT: no longer R1.1
Changed lines of the file:
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@@
 <part name="GND2" library="supply1" deviceset="GND" device=""/>
 <part name="SW1" library="dp_devices" deviceset="SW_TACT_4P" device=""/>
-<part name="R1" library="rcl" deviceset="R-US_" device="R0805" value="4K7"/>
 <part name="C1" library="rcl" deviceset="C-US" device="C0805" value="1uF"/>
 </parts>
@@
 <instance part="GND2" gate="1" x="68.58" y="27.94"/>
 <instance part="SW1" gate="G$1" x="68.58" y="43.18"/>
-<instance part="R1" gate="G$1" x="63.5" y="78.74"/>
 <instance part="C1" gate="G$1" x="5.08" y="63.5"/>
 </instances>
@@
 <wire x1="83.82" y1="78.74" x2="73.66" y2="78.74" width="0.1524" layer="91"/>
 <wire x1="73.66" y1="78.74" x2="73.66" y2="86.36" width="0.1524" layer="91"/>
-<pinref part="R1" gate="G$1" pin="2"/>
-<wire x1="68.58" y1="78.74" x2="73.66" y2="78.74" width="0.1524" layer="91"/>
-<junction x="73.66" y="78.74"/>
 </segment>
 </net>
@@
 <pinref part="U1" gate="G$1" pin="PB3(ADC3)"/>
 <wire x1="43.18" y1="66.04" x2="55.88" y2="66.04" width="0.1524" layer="91"/>
-<pinref part="R1" gate="G$1" pin="1"/>
-<wire x1="55.88" y1="66.04" x2="55.88" y2="78.74" width="0.1524" layer="91"/>
-<wire x1="55.88" y1="78.74" x2="58.42" y2="78.74" width="0.1524" layer="91"/>
 <wire x1="55.88" y1="66.04" x2="60.96" y2="66.04" width="0.1524" layer="91"/>
-<junction x="55.88" y="66.04"/>
 <wire x1="60.96" y1="66.04" x2="60.96" y2="43.18" width="0.1524" layer="91"/>
 <pinref part="SW1" gate="G$1" pin="1"/>

Commit message: osh-2: fix swapped MOSFET drain/source
Parts:
- JP1: value (none) -> IN
- JP2: value (none) -> OUT
- SW1: value (none) -> USER
Connections:
- net GND: now also Q1.S; no longer Q1.D
- net PWM_VSS: now also Q1.D; no longer Q1.S
Other:
- moved on the sheet: Q1, SW1
Changed lines of the file:
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@@
 <part name="U1" library="SparkFun-DigitalIC" deviceset="ATTINY45" device="TINY85-20-SMT" value="Tiny85-20-SMT"/>
 <part name="ICSP" library="Protofusion" deviceset="POGOPIN-CONN" device="WITHVIAS"/>
-<part name="JP1" library="pinhead" deviceset="PINHD-1X2" device=""/>
-<part name="JP2" library="pinhead" deviceset="PINHD-1X2" device=""/>
+<part name="JP1" library="pinhead" deviceset="PINHD-1X2" device="" value="IN"/>
+<part name="JP2" library="pinhead" deviceset="PINHD-1X2" device="" value="OUT"/>
 <part name="P+1" library="supply1" deviceset="+5V" device=""/>
 <part name="P+2" library="supply1" deviceset="+5V" device=""/>
 <part name="GND1" library="supply1" deviceset="GND" device=""/>
 <part name="GND2" library="supply1" deviceset="GND" device=""/>
-<part name="SW1" library="dp_devices" deviceset="SW_TACT_4P" device=""/>
+<part name="SW1" library="dp_devices" deviceset="SW_TACT_4P" device="" value="USER"/>
 <part name="C1" library="rcl" deviceset="C-US" device="C0805" value="1uF"/>
 </parts>
@@
 </plain>
 <instances>
-<instance part="Q1" gate="G$1" x="68.58" y="58.42" rot="R90"/>
+<instance part="Q1" gate="G$1" x="71.12" y="66.04"/>
 <instance part="U1" gate="G$1" x="30.48" y="66.04"/>
 <instance part="ICSP" gate="J" x="-10.16" y="45.72" rot="R180"/>
@@
 <instance part="GND1" gate="1" x="12.7" y="27.94"/>
 <instance part="GND2" gate="1" x="68.58" y="27.94"/>
-<instance part="SW1" gate="G$1" x="68.58" y="43.18"/>
+<instance part="SW1" gate="G$1" x="63.5" y="43.18"/>
 <instance part="C1" gate="G$1" x="5.08" y="63.5"/>
 </instances>
@@
 <wire x1="48.26" y1="73.66" x2="43.18" y2="73.66" width="0.1524" layer="91"/>
 <pinref part="Q1" gate="G$1" pin="G"/>
-<wire x1="71.12" y1="55.88" x2="71.12" y2="53.34" width="0.1524" layer="91"/>
-<wire x1="71.12" y1="53.34" x2="58.42" y2="53.34" width="0.1524" layer="91"/>
-<wire x1="58.42" y1="53.34" x2="58.42" y2="73.66" width="0.1524" layer="91"/>
+<wire x1="68.58" y1="63.5" x2="58.42" y2="63.5" width="0.1524" layer="91"/>
+<wire x1="58.42" y1="63.5" x2="58.42" y2="73.66" width="0.1524" layer="91"/>
 <wire x1="58.42" y1="73.66" x2="48.26" y2="73.66" width="0.1524" layer="91"/>
 <junction x="48.26" y="73.66"/>
@@
 <net name="GND" class="0">
 <segment>
-<pinref part="Q1" gate="G$1" pin="D"/>
-<wire x1="63.5" y1="60.96" x2="55.88" y2="60.96" width="0.1524" layer="91"/>
-<wire x1="55.88" y1="60.96" x2="55.88" y2="35.56" width="0.1524" layer="91"/>
 <pinref part="GND1" gate="1" pin="GND"/>
 <wire x1="55.88" y1="35.56" x2="12.7" y2="35.56" width="0.1524" layer="91"/>
@@
 <wire x1="68.58" y1="35.56" x2="68.58" y2="30.48" width="0.1524" layer="91"/>
 <wire x1="55.88" y1="35.56" x2="68.58" y2="35.56" width="0.1524" layer="91"/>
-<junction x="55.88" y="35.56"/>
-<wire x1="68.58" y1="35.56" x2="76.2" y2="35.56" width="0.1524" layer="91"/>
-<wire x1="76.2" y1="35.56" x2="76.2" y2="40.64" width="0.1524" layer="91"/>
+<wire x1="68.58" y1="35.56" x2="71.12" y2="35.56" width="0.1524" layer="91"/>
+<wire x1="71.12" y1="35.56" x2="71.12" y2="40.64" width="0.1524" layer="91"/>
 <junction x="68.58" y="35.56"/>
 <pinref part="SW1" gate="G$1" pin="3"/>
-<wire x1="76.2" y1="40.64" x2="76.2" y2="43.18" width="0.1524" layer="91"/>
-<wire x1="76.2" y1="43.18" x2="73.66" y2="43.18" width="0.1524" layer="91"/>
+<wire x1="71.12" y1="40.64" x2="71.12" y2="43.18" width="0.1524" layer="91"/>
+<wire x1="71.12" y1="43.18" x2="68.58" y2="43.18" width="0.1524" layer="91"/>
 <pinref part="SW1" gate="G$1" pin="4"/>
-<wire x1="73.66" y1="40.64" x2="76.2" y2="40.64" width="0.1524" layer="91"/>
-<junction x="76.2" y="40.64"/>
+<wire x1="68.58" y1="40.64" x2="71.12" y2="40.64" width="0.1524" layer="91"/>
+<junction x="71.12" y="40.64"/>
+<pinref part="Q1" gate="G$1" pin="S"/>
+<wire x1="73.66" y1="60.96" x2="73.66" y2="35.56" width="0.1524" layer="91"/>
+<wire x1="73.66" y1="35.56" x2="71.12" y2="35.56" width="0.1524" layer="91"/>
+<junction x="71.12" y="35.56"/>
 </segment>
 </net>
@@
 <pinref part="JP2" gate="G$1" pin="2"/>
 <wire x1="83.82" y1="76.2" x2="76.2" y2="76.2" width="0.1524" layer="91"/>
-<wire x1="76.2" y1="76.2" x2="76.2" y2="60.96" width="0.1524" layer="91"/>
-<wire x1="76.2" y1="60.96" x2="73.66" y2="60.96" width="0.1524" layer="91"/>
-<pinref part="Q1" gate="G$1" pin="S"/>
+<wire x1="76.2" y1="76.2" x2="73.66" y2="76.2" width="0.1524" layer="91"/>
+<wire x1="73.66" y1="76.2" x2="73.66" y2="71.12" width="0.1524" layer="91"/>
+<pinref part="Q1" gate="G$1" pin="D"/>
 </segment>
 </net>
@@
 <pinref part="U1" gate="G$1" pin="PB3(ADC3)"/>
 <wire x1="43.18" y1="66.04" x2="55.88" y2="66.04" width="0.1524" layer="91"/>
-<wire x1="55.88" y1="66.04" x2="60.96" y2="66.04" width="0.1524" layer="91"/>
-<wire x1="60.96" y1="66.04" x2="60.96" y2="43.18" width="0.1524" layer="91"/>
+<wire x1="55.88" y1="66.04" x2="55.88" y2="43.18" width="0.1524" layer="91"/>
+<pinref part="SW1" gate="G$1" pin="2"/>
+<wire x1="55.88" y1="43.18" x2="55.88" y2="40.64" width="0.1524" layer="91"/>
+<wire x1="58.42" y1="40.64" x2="55.88" y2="40.64" width="0.1524" layer="91"/>
 <pinref part="SW1" gate="G$1" pin="1"/>
-<wire x1="60.96" y1="43.18" x2="63.5" y2="43.18" width="0.1524" layer="91"/>
-<pinref part="SW1" gate="G$1" pin="2"/>
-<wire x1="63.5" y1="40.64" x2="60.96" y2="40.64" width="0.1524" layer="91"/>
-<wire x1="60.96" y1="40.64" x2="60.96" y2="43.18" width="0.1524" layer="91"/>
-<junction x="60.96" y="43.18"/>
+<wire x1="58.42" y1="43.18" x2="55.88" y2="43.18" width="0.1524" layer="91"/>
+<junction x="55.88" y="43.18"/>
 </segment>
 </net>
@@
 </sheet>
 </sheets>
-<errors>
-</errors>
 </schematic>
 </drawing>
